File: hardware/KiCad/tentacle-mini.kicad_pcb (KiCad board)
At the start: 2 copper layers, 68.6 x 53.3 mm, 36 parts, among them P1 BNC, P2 BNC, SW1 SW_PUSH

Commit message: Update for KiCad v4
Parts:
- C1, C10, C2, C3, C4, C5, C6, C7, C8, C9, R1, R2, R3, R4, R5, R6: footprint SM0805a -> tentacle:SM0805a
- C11: footprint c_tant_X -> tentacle:c_tant_X
- DCDC1, DCDC2: footprint R1SE_0505 -> tentacle:R1SE_0505
- P1, P2: footprint BNC-1337543a -> tentacle:BNC-1337543a
- REG1, REG2: footprint sot89a -> tentacle:sot89a
- SHIELD1: footprint ARDUINO_SHIELD_040pinsb_no_outline -> tentacle:ARDUINO_SHIELD_040pinsb_no_outline
- SIG_ISO1, SIG_ISO2: footprint so-8a -> tentacle:so-8a
- STP1, STP2: footprint Atlas_Stamp_14x21 -> tentacle:Atlas_Stamp_14x21
- SW1: footprint B3S-1000P -> tentacle:B3S-1000P
