File: hardware/KiCad/tentacle-mini.sch (KiCad schematic (older format))
At the start: 29 parts, among them P1 BNC, P2 BNC, SW1 SW_PUSH

Commit message: Update for KiCad v4
Parts:
- C1, C10, C2, C3, C4, C5, C6, C7, C8, C9, R1, R2, R3, R4, R5, R6: footprint ~ -> tentacle:SM0805a
- C11: footprint ~ -> tentacle:c_tant_X
- DCDC1, DCDC2: footprint ~ -> tentacle:R1SE_0505
- P1, P2: footprint ~ -> tentacle:BNC-1337543a
- REG1, REG2: footprint ~ -> tentacle:sot89a
- SHIELD1: footprint (none) -> tentacle:ARDUINO_SHIELD_040pinsb_no_outline
- SIG_ISO1, SIG_ISO2: footprint ~ -> tentacle:so-8a
- STP1, STP2: footprint ~ -> tentacle:Atlas_Stamp_14x21
- SW1: footprint ~ -> tentacle:B3S-1000P
Changed lines of the file:
@@
 EESchema Schematic File Version 2
+LIBS:tentacle-mini
 LIBS:power
 LIBS:device
@@
 LIBS:memory
 LIBS:xilinx
-LIBS:special
 LIBS:microcontrollers
 LIBS:dsp
@@
 LIBS:contrib
 LIBS:valves
-LIBS:tentacle-mini
 LIBS:tentacle-mini-cache
-EELAYER 27 0
+EELAYER 25 0
 EELAYER END
 $Descr A3 16535 11693
@@
 F 0 "SIG_ISO2" H 9300 2250 60  0000 C CNN
 F 1 "SI8600" V 8950 2900 60  0000 C CNN
-F 2 "~" H 8900 2850 60  0000 C CNN
+F 2 "tentacle:so-8a" H 8900 2850 60  0001 C CNN
 F 3 "~" H 8900 2850 60  0000 C CNN
 	1    8900 2850
@@
 F 0 "SIG_ISO1" H 6400 2250 60  0000 C CNN
 F 1 "SI8600" V 6050 2900 60  0000 C CNN
-F 2 "~" H 6000 2850 60  0000 C CNN
+F 2 "tentacle:so-8a" H 6000 2850 60  0001 C CNN
 F 3 "~" H 6000 2850 60  0000 C CNN
 	1    6000 2850
@@
 F 0 "STP1" H 6300 5650 60  0000 C CNN
 F 1 "ATLAS_STAMP" H 5850 6350 60  0000 C CNN
-F 2 "~" H 5850 7100 60  0000 C CNN
+F 2 "tentacle:Atlas_Stamp_14x21" H 5850 7100 60  0001 C CNN
 F 3 "~" H 5850 7100 60  0000 C CNN
 	1    5850 6100
@@
 F 0 "STP2" H 9200 5650 60  0000 C CNN
 F 1 "ATLAS_STAMP" H 8750 6350 60  0000 C CNN
-F 2 "~" H 8750 7100 60  0000 C CNN
+F 2 "tentacle:Atlas_Stamp_14x21" H 8750 7100 60  0001 C CNN
 F 3 "~" H 8750 7100 60  0000 C CNN
 	1    8750 6100
@@
 F 0 "SW1" H 12300 4760 50  0000 C CNN
 F 1 "SW_PUSH" H 12150 4570 50  0000 C CNN
-F 2 "~" H 12150 4650 60  0000 C CNN
+F 2 "tentacle:B3S-1000P" H 12150 4650 60  0001 C CNN
 F 3 "~" H 12150 4650 60  0000 C CNN
 	1    12150 4650
@@
 F 0 "P1" H 6110 7520 60  0000 C CNN
 F 1 "BNC" V 6210 7340 40  0000 C CNN
-F 2 "~" H 6100 7400 60  0000 C CNN
+F 2 "tentacle:BNC-1337543a" H 6100 7400 60  0001 C CNN
 F 3 "~" H 6100 7400 60  0000 C CNN
 	1    6100 7400
@@
 F 0 "P2" H 9010 7520 60  0000 C CNN
 F 1 "BNC" V 9110 7340 40  0000 C CNN
-F 2 "~" H 9000 7400 60  0000 C CNN
+F 2 "tentacle:BNC-1337543a" H 9000 7400 60  0001 C CNN
 F 3 "~" H 9000 7400 60  0000 C CNN
 	1    9000 7400
@@
 F 0 "C5" H 5450 1850 40  0000 L CNN
 F 1 "0.1 µF" H 5350 1650 40  0000 L CNN
-F 2 "~" H 5488 1600 30  0000 C CNN
+F 2 "tentacle:SM0805a" H 5488 1600 30  0001 C CNN
 F 3 "~" H 5450 1750 60  0000 C CNN
 	1    5450 1750
@@
 F 0 "C10" H 8350 1850 40  0000 L CNN
 F 1 "0.1 µF" H 8250 1650 40  0000 L CNN
-F 2 "~" H 8388 1600 30  0000 C CNN
+F 2 "tentacle:SM0805a" H 8388 1600 30  0001 C CNN
 F 3 "~" H 8350 1750 60  0000 C CNN
 	1    8350 1750
@@
 F 0 "DCDC1" H 6200 7800 60  0000 C CNN
 F 1 "R1SE_0505" V 5900 8400 60  0000 C CNN
-F 2 "~" H 5750 7950 60  0000 C CNN
+F 2 "tentacle:R1SE_0505" H 5750 7950 60  0001 C CNN
 F 3 "~" H 5750 7950 60  0000 C CNN
 	1    5900 8300
@@
 F 0 "R1" V 6080 4000 40  0000 C CNN
 F 1 "4.7K" V 6007 4001 40  0000 C CNN
-F 2 "~" V 5930 4000 30  0000 C CNN
+F 2 "tentacle:SM0805a" V 5930 4000 30  0001 C CNN
 F 3 "~" H 6000 4000 30  0000 C CNN
 	1    6000 4000
@@
 F 0 "R2" V 5830 3950 40  0000 C CNN
 F 1 "4.7K" V 5757 3951 40  0000 C CNN
-F 2 "~" V 5680 3950 30  0000 C CNN
+F 2 "tentacle:SM0805a" V 5680 3950 30  0001 C CNN
 F 3 "~" H 5750 3950 30  0000 C CNN
 	1    5750 3950
@@
 F 0 "R3" V 8980 4000 40  0000 C CNN
 F 1 "4.7K" V 8907 4001 40  0000 C CNN
-F 2 "~" V 8830 4000 30  0000 C CNN
+F 2 "tentacle:SM0805a" V 8830 4000 30  0001 C CNN
 F 3 "~" H 8900 4000 30  0000 C CNN
 	1    8900 4000
@@
 F 0 "R4" V 8730 3950 40  0000 C CNN
 F 1 "4.7K" V 8657 3951 40  0000 C CNN
-F 2 "~" V 8580 3950 30  0000 C CNN
+F 2 "tentacle:SM0805a" V 8580 3950 30  0001 C CNN
 F 3 "~" H 8650 3950 30  0000 C CNN
 	1    8650 3950
@@
 F 0 "C4" H 5350 3900 40  0000 L CNN
 F 1 "0.1 µF" H 5250 3700 40  0000 L CNN
-F 2 "~" H 5388 3650 30  0000 C CNN
+F 2 "tentacle:SM0805a" H 5388 3650 30  0001 C CNN
 F 3 "~" H 5350 3800 60  0000 C CNN
 	1    5350 3800
@@
 F 0 "C9" H 8300 3900 40  0000 L CNN
 F 1 "0.1 µF" H 8200 3700 40  0000 L CNN
-F 2 "~" H 8338 3650 30  0000 C CNN
+F 2 "tentacle:SM0805a" H 8338 3650 30  0001 C CNN
 F 3 "~" H 8300 3800 60  0000 C CNN
 	1    8300 3800
@@
 F 0 "C2" H 5850 9150 40  0000 L CNN
 F 1 "1µF" H 5856 8965 40  0000 L CNN
-F 2 "~" H 5888 8900 30  0000 C CNN
+F 2 "tentacle:SM0805a" H 5888 8900 30  0001 C CNN
 F 3 "~" H 5850 9050 60  0000 C CNN
 	1    5850 9050
@@
 F 0 "C3" H 6700 10400 40  0000 L CNN
 F 1 "2.2µF" H 6706 10215 40  0000 L CNN
-F 2 "~" H 6738 10150 30  0000 C CNN
+F 2 "tentacle:SM0805a" H 6738 10150 30  0001 C CNN
 F 3 "~" H 6700 10300 60  0000 C CNN
 	1    6700 10300
@@
 F 0 "DCDC2" H 9100 7800 60  0000 C CNN
 F 1 "R1SE_0505" V 8800 8400 60  0000 C CNN
-F 2 "~" H 8650 7950 60  0000 C CNN
+F 2 "tentacle:R1SE_0505" H 8650 7950 60  0001 C CNN
 F 3 "~" H 8650 7950 60  0000 C CNN
 	1    8800 8300
@@
 F 0 "C7" H 8750 9150 40  0000 L CNN
 F 1 "1µF" H 8756 8965 40  0000 L CNN
-F 2 "~" H 8788 8900 30  0000 C CNN
+F 2 "tentacle:SM0805a" H 8788 8900 30  0001 C CNN
 F 3 "~" H 8750 9050 60  0000 C CNN
 	1    8750 9050
@@
 F 0 "C8" H 9600 10400 40  0000 L CNN
 F 1 "2.2µF" H 9606 10215 40  0000 L CNN
-F 2 "~" H 9638 10150 30  0000 C CNN
+F 2 "tentacle:SM0805a" H 9638 10150 30  0001 C CNN
 F 3 "~" H 9600 10300 60  0000 C CNN
 	1    9600 10300
@@
 F 0 "REG1" H 6150 9300 60  0000 C CNN
 F 1 "LD2981ABU50TR" H 5750 10400 60  0000 C CNN
-F 2 "~" H 5800 9850 60  0000 C CNN
+F 2 "tentacle:sot89a" H 5800 9850 60  0001 C CNN
 F 3 "~" H 5800 9850 60  0000 C CNN
 	1    5800 9850
@@
 F 0 "REG2" H 9050 9300 60  0000 C CNN
 F 1 "LD2981ABU50TR" H 8650 10400 60  0000 C CNN
-F 2 "~" H 8700 9850 60  0000 C CNN
+F 2 "tentacle:sot89a" H 8700 9850 60  0001 C CNN
 F 3 "~" H 8700 9850 60  0000 C CNN
 	1    8700 9850
@@
 F 0 "C1" H 5400 7150 40  0000 L CNN
 F 1 "1µF" H 5406 6965 40  0000 L CNN
-F 2 "~" H 5438 6900 30  0000 C CNN
+F 2 "tentacle:SM0805a" H 5438 6900 30  0001 C CNN
 F 3 "~" H 5400 7050 60  0000 C CNN
 	1    5400 7050
@@
 F 0 "C6" H 8300 7150 40  0000 L CNN
 F 1 "1µF" H 8306 6965 40  0000 L CNN
-F 2 "~" H 8338 6900 30  0000 C CNN
+F 2 "tentacle:SM0805a" H 8338 6900 30  0001 C CNN
 F 3 "~" H 8300 7050 60  0000 C CNN
 	1    8300 7050
@@
 F 0 "R6" V 11030 2100 40  0000 C CNN
 F 1 "4.7K" V 10957 2101 40  0000 C CNN
-F 2 "~" V 10880 2100 30  0000 C CNN
+F 2 "tentacle:SM0805a" V 10880 2100 30  0001 C CNN
 F 3 "~" H 10950 2100 30  0000 C CNN
 	1    10950 2100
@@
 F 0 "R5" V 10830 2100 40  0000 C CNN
 F 1 "4.7K" V 10757 2101 40  0000 C CNN
-F 2 "~" V 10680 2100 30  0000 C CNN
+F 2 "tentacle:SM0805a" V 10680 2100 30  0001 C CNN
 F 3 "~" H 10750 2100 30  0000 C CNN
 	1    10750 2100
@@
 F 0 "SHIELD1" H 12500 4350 60  0000 C CNN
 F 1 "ARDUINO_SHIELD" H 12900 2450 60  0000 C CNN
-F 2 "" H 12850 3400 60  0000 C CNN
+F 2 "tentacle:ARDUINO_SHIELD_040pinsb_no_outline" H 12850 3400 60  0001 C CNN
 F 3 "" H 12850 3400 60  0000 C CNN
 	1    12850 3400
@@
 F 0 "C11" H 12750 5450 50  0000 L CNN
 F 1 "470µF" H 12750 5250 50  0000 L CNN
-F 2 "~" H 12700 5350 60  0000 C CNN
+F 2 "tentacle:c_tant_X" H 12700 5350 60  0001 C CNN
 F 3 "~" H 12700 5350 60  0000 C CNN
 	1    12700 5350
@@
 Connection ~ 5600 3600
 $Comp
-L VCOM #PWR13
+L VCOM #PWR030
 U 1 1 56613AB1
 P 11900 4400
-F 0 "#PWR13" H 11900 4600 40  0001 C CNN
+F 0 "#PWR030" H 11900 4600 40  0001 C CNN
 F 1 "VCOM" H 11900 4550 40  0000 C CNN
 F 2 "" H 11900 4400 60  0000 C CNN
@@
 	11900 4450 11900 4400
 $Comp
-L VCOM #PWR4
+L VCOM #PWR031
 U 1 1 56613BF5
 P 5650 1700
-F 0 "#PWR4" H 5650 1900 40  0001 C CNN
+F 0 "#PWR031" H 5650 1900 40  0001 C CNN
 F 1 "VCOM" H 5650 1850 40  0000 C CNN
 F 2 "" H 5650 1700 60  0000 C CNN
@@
 $EndComp
 $Comp
-L VCOM #PWR9
+L VCOM #PWR032
 U 1 1 56613C04
 P 8550 1700
-F 0 "#PWR9" H 8550 1900 40  0001 C CNN
+F 0 "#PWR032" H 8550 1900 40  0001 C CNN
 F 1 "VCOM" H 8550 1850 40  0000 C CNN
 F 2 "" H 8550 1700 60  0000 C CNN
@@
 $EndComp
 $Comp
-L VCOM #PWR11
+L VCOM #PWR033
 U 1 1 5661271B
 P 10850 2600
-F 0 "#PWR11" H 10850 2800 40  0001 C CNN
+F 0 "#PWR033" H 10850 2800 40  0001 C CNN
 F 1 "VCOM" H 10850 2750 40  0000 C CNN
 F 2 "" H 10850 2600 60  0000 C CNN
